File: RainLight.kicad_sch (KiCad schematic)
At the start: 21 parts, among them J1 DTM04-2P (wire pigtail)

Commit message: Swap resistors to flat/horizontal 7.62mm footprint
Parts:
- D1, D10, D2, D3, D4, D5, D6, D7, D8, D9: KiLib_Generator (none) -> LED/THT
- J1: KiLib_Generator (none) -> connector/wire
Connections:
- net VCC: now also J1.1 (Pin_1), J1.2 (Pin_2)

Commit message: Update R1-R10 from 1.2k to 510 ohm
Based on confirmed LED spec (Chanzon 10mm red, Vf=2.0V @ 20mA) at 12V
source: R = (12-2)/0.02 = 500 ohm, rounded to nearest standard value (510).
Value-only change - footprint/wattage unchanged, still the 1/4W-sized
DIN0207 axial package. Actual dissipation at 510ohm/20mA is ~0.2W, close
to the 1/4W package's rating - a genuine 1/2W part would need a larger
footprint (not yet done, pending a real part number).
Parts:
- R1, R10, R2, R3, R4, R5, R6, R7, R8, R9: value 1.2k -> 510
Changed lines of the file:
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@@
 			)
 		)
-		(property "Value" "1.2k"
+		(property "Value" "510"
 			(at 88.9 54.61 90)
 			(show_name no)
@@
 			)
 		)
-		(property "Value" "1.2k"
+		(property "Value" "510"
 			(at 88.9 168.91 90)
 			(show_name no)
@@
 			)
 		)
-		(property "Value" "1.2k"
+		(property "Value" "510"
 			(at 88.9 105.41 90)
 			(show_name no)
@@
 			)
 		)
-		(property "Value" "1.2k"
+		(property "Value" "510"
 			(at 88.9 143.51 90)
 			(show_name no)
@@
 			)
 		)
-		(property "Value" "1.2k"
+		(property "Value" "510"
 			(at 88.9 92.71 90)
 			(show_name no)
@@
 			)
 		)
-		(property "Value" "1.2k"
+		(property "Value" "510"
 			(at 88.9 118.11 90)
 			(show_name no)
@@
 			)
 		)
-		(property "Value" "1.2k"
+		(property "Value" "510"
 			(at 88.9 130.81 90)
 			(show_name no)
@@
 			)
 		)
-		(property "Value" "1.2k"
+		(property "Value" "510"
 			(at 88.9 67.31 90)
 			(show_name no)
@@
 			)
 		)
-		(property "Value" "1.2k"
+		(property "Value" "510"
 			(at 88.9 156.21 90)
 			(show_name no)
@@
 			)
 		)
-		(property "Value" "1.2k"
+		(property "Value" "510"
 			(at 88.9 80.01 90)
 			(show_name no)
